File: uBraids_SE_Assembly_Template.brd (EAGLE design)
At the start: 40 x 110.5 mm, 0 parts

Commit message: Revision F
Parts:
- added E$1, E$2, E$3: (no value), uBraids_SE_Library:M2.5-HOLE
Routing:
- added copper zone on layer 1, net GND
- added copper zone on layer 16, net GND
Other:
- board text added: "2.0 mm"
- board text added: "µBraids SE Assembly Template TD-UBSE-F-AT CC BY-SA 4.0 2020-02-08 tall-dog.com"
- board text removed: "µBraids SE Assembly Template TD-UBSE-E-AT CC BY-SA 4.0 2018-04-28 tall-dog.com"
Changed lines of the file:
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@@
 <?xml version="1.0" encoding="utf-8"?>
 <!DOCTYPE eagle SYSTEM "eagle.dtd">
-<eagle version="9.0.0">
+<eagle version="9.5.2">
 <drawing>
 <settings>
@@
 <layer number="51" name="tDocu" color="7" fill="1" visible="yes" active="yes"/>
 <layer number="52" name="bDocu" color="7" fill="1" visible="yes" active="yes"/>
+<layer number="88" name="SimResults" color="9" fill="1" visible="no" active="no"/>
+<layer number="89" name="SimProbes" color="9" fill="1" visible="no" active="no"/>
+<layer number="90" name="Modules" color="5" fill="1" visible="no" active="no"/>
+<layer number="91" name="Nets" color="2" fill="1" visible="no" active="no"/>
+<layer number="92" name="Busses" color="1" fill="1" visible="no" active="no"/>
+<layer number="93" name="Pins" color="2" fill="1" visible="no" active="no"/>
+<layer number="94" name="Symbols" color="4" fill="1" visible="no" active="no"/>
+<layer number="95" name="Names" color="7" fill="1" visible="no" active="no"/>
+<layer number="96" name="Values" color="7" fill="1" visible="no" active="no"/>
+<layer number="97" name="Info" color="7" fill="1" visible="no" active="no"/>
+<layer number="98" name="Guide" color="6" fill="1" visible="no" active="no"/>
 </layers>
 <board>
 <plain>
-<text x="20.5" y="102" size="3" layer="21" ratio="10" rot="R180" align="center">THIS SIDE
+<text x="20.5" y="102" size="3" layer="21" ratio="14" rot="R180" align="center">THIS SIDE
 FACES UP</text>
 <wire x1="37" y1="110.5" x2="3" y2="110.5" width="0" layer="20"/>
@@
 <hole x="32.5" y="12" drill="6.2"/>
 <hole x="20" y="4.5" drill="6.2"/>
-<text x="20" y="86" size="2" layer="21" align="center">µBraids SE
+<text x="20" y="86" size="2" layer="21" ratio="12" align="center">µBraids SE
 Assembly Template
-TD-UBSE-E-AT
+TD-UBSE-F-AT
 CC BY-SA 4.0
-2018-04-28
+2020-02-08
 tall-dog.com</text>
-<text x="20" y="86" size="2" layer="22" rot="MR0" align="center">µBraids SE
+<text x="20" y="86" size="2" layer="22" ratio="12" rot="MR0" align="center">µBraids SE
 Assembly Template
-TD-UBSE-E-AT
+TD-UBSE-F-AT
 CC BY-SA 4.0
-2018-04-28
+2020-02-08
 tall-dog.com</text>
-<text x="20.5" y="102" size="3" layer="22" ratio="10" rot="MR180" align="center">THIS SIDE
+<text x="20.5" y="102" size="3" layer="22" ratio="14" rot="MR180" align="center">THIS SIDE
 FACES DOWN</text>
+<text x="20" y="49.5" size="3.5" layer="22" ratio="12" rot="MR0" align="center">2.0 mm</text>
+<text x="20" y="49.5" size="3.5" layer="21" ratio="12" align="center">2.0 mm</text>
+<wire x1="12" y1="52.5" x2="28" y2="52.5" width="0.254" layer="21"/>
+<wire x1="28" y1="52.5" x2="28" y2="46.5" width="0.254" layer="21"/>
+<wire x1="28" y1="46.5" x2="12" y2="46.5" width="0.254" layer="21"/>
+<wire x1="12" y1="46.5" x2="12" y2="52.5" width="0.254" layer="21"/>
+<wire x1="12" y1="52.5" x2="28" y2="52.5" width="0.254" layer="22"/>
+<wire x1="28" y1="52.5" x2="28" y2="46.5" width="0.254" layer="22"/>
+<wire x1="28" y1="46.5" x2="12" y2="46.5" width="0.254" layer="22"/>
+<wire x1="12" y1="46.5" x2="12" y2="52.5" width="0.254" layer="22"/>
 </plain>
 <attributes>
@@
 <param name="checkStop" value="0"/>
 <param name="checkValues" value="0"/>
+<param name="checkNames" value="1"/>
+<param name="checkWireStubs" value="1"/>
+<param name="checkPolygonWidth" value="0"/>
 <param name="useDiameter" value="13"/>
 <param name="maxErrors" value="50"/>
@@
 </autorouter>
 <elements>
+<element name="E$1" library="uBraids_SE_Library" package="M2.5-HOLE" value="" x="3" y="107.5" smashed="yes"/>
+<element name="E$2" library="uBraids_SE_Library" package="M2.5-HOLE" value="" x="37" y="107.5" smashed="yes"/>
+<element name="E$3" library="uBraids_SE_Library" package="M2.5-HOLE" value="" x="3" y="3" smashed="yes"/>
 </elements>
 <signals>
-<signal name="S$1">
-<via x="3" y="107.5" extent="1-16" drill="2.75" diameter="5"/>
-</signal>
-<signal name="S$2">
-<via x="37" y="107.5" extent="1-16" drill="2.75" diameter="5"/>
-</signal>
-<signal name="S$3">
-<via x="3" y="3" extent="1-16" drill="2.75" diameter="5"/>
+<signal name="GND">
+<polygon width="0.5" layer="1" isolate="0.5">
+<vertex x="0" y="110.5"/>
+<vertex x="40" y="110.5"/>
+<vertex x="40" y="0"/>
+<vertex x="0" y="0"/>
+</polygon>
+<polygon width="0.5" layer="16" isolate="0.5">
+<vertex x="0" y="110.5"/>
+<vertex x="40" y="110.5"/>
+<vertex x="40" y="0"/>
+<vertex x="0" y="0"/>
+</polygon>
 </signal>
 </signals>
+<mfgpreviewcolors>
+<mfgpreviewcolor name="soldermaskcolor" color="0xC8008000"/>
+<mfgpreviewcolor name="silkscreencolor" color="0xFFFEFEFE"/>
+<mfgpreviewcolor name="backgroundcolor" color="0xFF282828"/>
+<mfgpreviewcolor name="coppercolor" color="0xFFFFBF00"/>
+<mfgpreviewcolor name="substratecolor" color="0xFF786E46"/>
+</mfgpreviewcolors>
+<errors>
+</errors>
 </board>
 </drawing>
