File: uBraids_SE_Main_Board.brd (EAGLE design)
At the start: 40 x 110.5 mm, 103 parts, among them J1 JACK-THONKICONN, J2 JACK-THONKICONN, J3 JACK-THONKICONN, J4 JACK-THONKICONN, J5 JACK-THONKICONN, J6 JACK-THONKICONN, P1 10kB, P2 10kB, P3 10kB, P4 10kB, P5 10kB, P6 10kB, Q1 MMBT3904, U1 STM32F103-LQFP-48, U2 DAC8551-VSSOP-8, U3 LM4040B25, U4 MCP3204-TSSOP-14, U5 LM1117-3.3, U6 LM4040B10, U7 MCP6004, U8 TL074-TSSOP-14, U9 TL072, X1 8MHz

Commit message: update for Revision E production
Parts:
- removed U$10: (no value), uBraids_SE:MARKING-OSH-LOGO-5MM
- removed U$15, U$16, U$9: (no value), uBraids_SE:FIDUCIAL
- removed U$4: (no value), uBraids_SE:MARKING-CC-BY-SA-4.0
- added HOLE3: HOLE, uBraids_SE_Library:M2.5-HOLE
- added P7: 10kB, uBraids_SE_Library:POT-ALP-VERT-PS
- added U$1, U$3, U$5: (no value), uBraids_SE_Library:FIDUCIAL
- added U$6: (no value), uBraids_SE_Library:MARKING-CC-LOGO
- added U$7: (no value), uBraids_SE_Library:MARKING-CC-BY-SA-4.0
- A1: device uBraids_SE:DISPLAY-MODULE -> uBraids_SE_Library:DISPLAY-MODULE
- C1, C10, C11, C14, C16, C17, C19, C2, C20, C21, C22, C23, C24, C25, C26, C27, C28, C29, C3, C30, C4, C5, C6, C7, C8, C9, R1, R10, R11, R12, R13, R14, R15, R16, R17, R18, R19, R2, R20, R21, R22, R23, R24, R25, R26, R27, R28, R29, R3, R30, R31, R32, R5, R6, R8, R9: device uBraids_SE:0603-NP -> uBraids_SE_Library:0603-NP
- C12, C13, C15, C18: device uBraids_SE:ELECTRO-SMD-6.6MM -> uBraids_SE_Library:ELECTRO-SMD-6.6MM
- C31: device uBraids_SE:ELECTRO-SMD-4.3MM -> uBraids_SE_Library:ELECTRO-SMD-4.3MM
- D1, D2: device uBraids_SE:SOD-123 -> uBraids_SE_Library:SOD-123
- H1: device uBraids_SE:PTH-0.05-2X5-SHROUDED-SMD -> uBraids_SE_Library:PTH-0.05-2X5-SHROUDED-SMD
- H2: device uBraids_SE:JST-XH-6 -> uBraids_SE_Library:JST-XH-6
- H3: device uBraids_SE:PTH-0.1-2X5-SHROUDED -> uBraids_SE_Library:PTH-0.1-2X5-SHROUDED
- HOLE1, HOLE2: device uBraids_SE:M2.5-HOLE -> uBraids_SE_Library:M2.5-HOLE
- J1, J2, J3, J4, J5, J6: device uBraids_SE:THONKICONN -> uBraids_SE_Library:THONKICONN
- P1, P2, P3, P4, P5, P6: device uBraids_SE:POT-ALP-VERT-PS -> uBraids_SE_Library:POT-ALP-VERT-PS
- Q1, U3, U6: device uBraids_SE:SOT-23 -> uBraids_SE_Library:SOT-23
- R4, R7: device uBraids_SE:0805-NP -> uBraids_SE_Library:0805-NP
- S1, S2: device uBraids_SE:BUTTON-EVQQ2 -> uBraids_SE_Library:BUTTON-EVQQ2
- S3: device uBraids_SE:ENCODER-EC12E -> uBraids_SE_Library:ENCODER-EC12E
- U$2: device uBraids_SE:MARKING-CC-LOGO -> uBraids_SE_Library:MARKING-OSH-LOGO-5MM
- U1: device uBraids_SE:LQFP-48 -> uBraids_SE_Library:LQFP-48
- U2: device uBraids_SE:VSSOP-8 -> uBraids_SE_Library:VSSOP-8
- U4, U7, U8: device uBraids_SE:TSSOP-14 -> uBraids_SE_Library:TSSOP-14
- U5: device uBraids_SE:WSON-8 -> uBraids_SE_Library:SOT-223
- U9: device uBraids_SE:TSSOP-8 -> uBraids_SE_Library:TSSOP-8
- X1: device uBraids_SE:CRYSTAL-ABM2 -> uBraids_SE_Library:CRYSTAL-ABM2
- moved U$2 15.2 mm to (25.5, 88.2)
- moved P4 14.6 mm to (20.0, 34.5)
- moved P5 14.6 mm to (32.5, 27.0)
- moved P6 14.6 mm to (20.0, 19.5)
- moved C14 4.72 mm to (23.2, 61.8), turned to 180 degrees
- moved C26 3.50 mm to (21.2, 19.8)
- moved U8 3.26 mm to (20.0, 23.5)
- moved R18 2.76 mm to (25.5, 27.0)
- moved C22 2.61 mm to (15.5, 29.5)
- moved C31 2.51 mm to (7.50, 6.50)
- moved C21 2.47 mm to (11.2, 35.5)
- moved R12 2.47 mm to (11.2, 37.2)
- moved R30 2.37 mm to (14.5, 7.50)
- moved R31 2.37 mm to (12.8, 7.50)
- moved R32 2.37 mm to (11.0, 7.50)
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Connections:
- removed net N$59: C23.1, P5.P$3, R19.1, R22.2, R23.2, U7.13
- new net N$1: P6.P$2, R26.2
- new net N$3: C23.1, P4.P$3, R19.1, R22.2, R23.2, U7.13
- net 12V_U5: no longer U5.2, U5.4
- net 3V3: now also U5.2, U5.4; no longer U5.5, U5.6, U5.7, U5.9
- net AREF_-10: now also P5.P$1, P7.P$1; no longer P4.P$1, P6.P$1
- net GND: now also P5.P$3, P7.P$3; no longer P4.P$3, P6.P$3
- net N$50: now also P4.P$1; no longer P5.P$1
- net N$61: now also P5.P$2; no longer P4.P$2
- net N$62: now also P4.P$2; no longer P5.P$2
- net N$63: now also P6.P$1; no longer R26.2
- net N$65: now also P7.P$2; no longer P6.P$2
- net N$70: now also P6.P$3
Routing:
- net N$59: track 47.9 -> 0.00 mm
- net N$3: track 0.00 -> 40.0 mm, vias 0 -> 2
- net N$1: track 0.00 -> 25.4 mm, vias 0 -> 3
- net N$70: track 44.3 -> 59.4 mm, vias 2 -> 3
- net N$63: track 31.4 -> 17.6 mm, vias 2 -> 1
- net N$62: track 8.08 -> 21.2 mm, vias 0 -> 1
- net 12V_U5: track 17.6 -> 9.52 mm
- net N$50: track 19.4 -> 11.4 mm, vias 0 -> 1
- net N$12: track 10.0 -> 13.8 mm
- net 12V: track 70.1 -> 73.8 mm
- net N$52: track 27.8 -> 31.1 mm
- net N$45: track 11.4 -> 14.7 mm
- net -12V: track 60.0 -> 63.1 mm
- net 3V3: track 175.5 -> 172.6 mm
- net N$67: track 21.1 -> 23.5 mm
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Other:
- board text added: "2018-04-27"
- board text added: "Board derived from work by Olivier Gillet of Mutable Instruments, Magpie Modular, and Neutron Sound"
- board text added: "TD-UBSE-E-MB"
- board text added: "µBraids SE Main Board TD-UBSE-E-MB CC BY-SA 4.0 2018-04-27 tall-dog.com"
- board text removed: "2017-12-29"
- board text removed: "Board derived from work by: Olivier Gillet of Mutable Instruments, Magpie Modular, and Neutron Sound"
- board text removed: "TD-UBSE-C"
- board text removed: "µBraids_SE TD-UBSE-C 2017-12-29 TALL-DOG.COM CC BY-SA 4.0"

Commit message: Revision F
Parts:
- removed S2: SPST-EVQQ2, uBraids_SE_Library:BUTTON-EVQQ2
- removed S3: ENCODER-SW, uBraids_SE_Library:ENCODER-EC12E
- removed U$5: (no value), uBraids_SE_Library:FIDUCIAL
- added C32: 10u, uBraids_SE_Library:ELECTRO-SMD-4.3MM
- added H4: HEADER-1X5-SSM, uBraids_SE_Library:SSM-105-S-SV-BE
- added H5: HEADER-2X5-PTH-0.1-SHROUDED, uBraids_SE_Library:PTH-0.1-2X5-SHROUDED
- added R33: 24.9k, uBraids_SE_Library:0603-NP
- added U$4: (no value), uBraids_SE_Library:LOGO-CC
- added U$8: (no value), uBraids_SE_Library:LOGO-OSHW
- A1: value DISPLAY-MODULE -> (none); device uBraids_SE_Library:DISPLAY-MODULE -> uBraids_SE_Library:DISPLAY-MODULE-OUTLINE
- C10, C17, C2, C26, C28, C3, C4, C5: value 100n -> 0.1u
- C11: value 470n -> 0.1u
- C12: value 22uF -> 22u
- C13: value 22uF -> 0.47u; device uBraids_SE_Library:ELECTRO-SMD-6.6MM -> uBraids_SE_Library:0603-NP
- C14: value 100n -> 22u; device uBraids_SE_Library:0603-NP -> uBraids_SE_Library:ELECTRO-SMD-6.6MM
- C15, C18: value 47uF -> 0.1u; device uBraids_SE_Library:ELECTRO-SMD-6.6MM -> uBraids_SE_Library:0603-NP
- C16: value 100n -> 47u; device uBraids_SE_Library:0603-NP -> uBraids_SE_Library:ELECTRO-SMD-6.6MM
- C19: value 1n -> 47u; device uBraids_SE_Library:0603-NP -> uBraids_SE_Library:ELECTRO-SMD-6.6MM
- C20, C22: value 100n -> 1n
- C21, C23, C29: value 1n -> 0.1u
- C24: value 100p -> 1n
- C25: value 100n -> 100p
- C30: value 47p -> 1n
- C31: value 10uF -> 47p; device uBraids_SE_Library:ELECTRO-SMD-4.3MM -> uBraids_SE_Library:0603-NP
- C6: value 18p -> 0.1u
- C7: value 1u -> 18p
- C8: value 100n -> 1u
- H1: value HEADER-2X5-PTH-0.05-SHROUDED-SMD -> HEADER-1X9-SSM; device uBraids_SE_Library:PTH-0.05-2X5-SHROUDED-SMD -> uBraids_SE_Library:SSM-109-S-SV-BE
- H2: value HEADER-1X6-PTH-SHROUDED -> HEADER-2X5-PTH-0.05-SHROUDED-SMD; device uBraids_SE_Library:JST-XH-6 -> uBraids_SE_Library:PTH-0.05-2X5-SHROUDED-SMD
- H3: value HEADER-2X5-PTH-0.1-SHROUDED -> HEADER-1X2; device uBraids_SE_Library:PTH-0.1-2X5-SHROUDED -> uBraids_SE_Library:PTH-0.1-1X2
- P1, P2, P3, P4, P5, P6, P7: device uBraids_SE_Library:POT-ALP-VERT-PS -> uBraids_SE_Library:POT
- R10, R18, R32: value 24.9k -> 100k
- R11: value 120k -> 200k
- R17, R25: value 100k -> 24.9k
- R19: value 49.9k -> 24.9k
- R2: value 10k -> 100R
- R20: value 39k -> 49.9k
- R21: value 24.9k -> 39k
- R27: value 49.9k -> 100k
- R28: value 24.9k -> 49.9k
- R29: value 200k -> 24.9k
- R3: value 1k -> 100R
- R30: value 1k -> 200k
- R31: value 100k -> 1k
- R4: value 4.7R -> 1k; device uBraids_SE_Library:0805-NP -> uBraids_SE_Library:0603-NP
- R7: value 330R -> 4.7R
- R8: value 100k -> 330R; device uBraids_SE_Library:0603-NP -> uBraids_SE_Library:0805-NP
- R9: value 200k -> 120k
- S1: value SPST-EVQQ2 -> ENCODER-SW; device uBraids_SE_Library:BUTTON-EVQQ2 -> uBraids_SE_Library:ENCODER-EC12E
- U$2: device uBraids_SE_Library:MARKING-OSH-LOGO-5MM -> uBraids_SE_Library:LOGO-REV
- U$3: device uBraids_SE_Library:FIDUCIAL -> uBraids_SE_Library:LOGO-OSH
- U$6: device uBraids_SE_Library:MARKING-CC-LOGO -> uBraids_SE_Library:FIDUCIAL
- U$7: device uBraids_SE_Library:MARKING-CC-BY-SA-4.0 -> uBraids_SE_Library:FIDUCIAL
- moved U$7 65.2 mm to (37.0, 3.00)
- moved U$6 47.9 mm to (4.00, 35.0)
- moved H3 40.1 mm to (2.50, 88.5)
- moved R27 30.1 mm to (2.50, 15.0)
- moved R8 29.1 mm to (29.0, 53.2), turned to 270 degrees
- moved C29 28.5 mm to (6.50, 17.2), turned to 270 degrees
- moved R20 27.6 mm to (30.5, 26.5), turned to 90 degrees
- moved C24 27.2 mm to (32.5, 26.5)
- moved R10 26.8 mm to (3.25, 39.8), turned to 180 degrees
- moved R21 24.5 mm to (3.00, 24.2), turned to 180 degrees
- moved C13 24.5 mm to (29.5, 76.0), turned to 270 degrees
- moved R14 23.8 mm to (10.5, 33.0), turned to 90 degrees
- moved S1 23.3 mm to (32.5, 72.0), flipped to the top, turned to 0 degrees
- moved C30 22.7 mm to (34.5, 12.0), turned to 90 degrees
- moved R11 22.3 mm to (33.5, 38.0), turned to 270 degrees
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Connections:
- removed net BOOT_FLASH: R1.2, S1.A1, S1.A2, U1.44
- removed net JTCK: H1.4, U1.37
- removed net JTDO: H1.6, U1.39
- removed net JTMS: H1.2, U1.34
- new net JTCK/SWCLK: H2.4, U1.37
- new net JTDO/SWO: H2.6, U1.39
- new net JTMS/SWDIO: H2.2, U1.34
- new net RX_R: R2.1, U1.31
- new net TX_R: R3.1, U1.30
- net -12V: now also C19.C, C29.2, D1.A, R8.1; no longer C18.C, C26.2, D2.A, R7.1
- net -12V_BUS: now also D1.C, H5.1, H5.2; no longer D2.C, H3.1, H3.2
- net 12V: now also C16.A, C23.1, C26.1, D2.C, R7.2; no longer C15.A, C22.1, C25.1, D1.C, R4.2
- net 12V_BUS: now also D2.A, H5.10, H5.9; no longer D1.A, H3.10, H3.9
- net 12V_U5: now also R7.1; no longer R4.1
- net 3V3: now also C11.1, C14.A, C15.1, C21.1, C6.1, H2.1, H4.1, R1.1, R4.1; no longer A1.5, C13.A, C14.1, C20.1, C4.1, C7.1, H1.1, R2.2, R3.1, S1.B1, S1.B2
- net AREF: now also C13.1, R4.2; no longer C11.1, R3.2
- net AREF_-10: now also C18.1, R11.1, R8.2; no longer C17.1, R7.2, R9.1
- net AUDIO_OUT: now also R21.2; no longer R20.2
- net DISP_CHAR1: now also H1.1; no longer A1.14
- net DISP_CHAR2: now also H1.2; no longer A1.13
- net DISP_CHAR3: now also H1.6; no longer A1.9
- net DISP_CHAR4: now also H1.9; no longer A1.6
- net DISP_EN: now also H4.5; no longer A1.1
- net DISP_SCK: now also H4.4; no longer A1.2
- net DISP_SER: now also H4.3; no longer A1.3
- net ENC_A: now also S1.B; no longer S3.B
- net ENC_B: now also S1.A; no longer S3.A
- net ENC_CLICK: now also S1.E; no longer S3.E
- net FINE_TUNE: now also C17.1; no longer C16.1
- net FM_CV: now also C20.2, R12.2; no longer C19.2, R10.2
- net GND: now also C13.2, C14.C, C15.2, C16.C, C18.2, C19.A, C21.2, C23.2, C26.2, C29.1, C6.2, C7.1, H1.4, H1.7, H1.8, H2.3, H2.5, H2.9, H4.2, H5.3, H5.4, H5.5, H5.6, H5.7, H5.8, S1.C, S1.D, U1.44; no longer A1.10, A1.11, A1.12, A1.4, A1.7, A1.8, C13.C, C14.2, C15.C, C16.2, C18.A, C20.2, C22.2, C24.2, C26.1, C6.1, C7.2, H1.9, H2.1, H3.3, H3.4, H3.5, H3.6, H3.7, H3.8, R1.1, S2.A1, S2.A2, S3.C, S3.D
- net JTDI: now also H2.8; no longer H1.8
- net N$1: now also R27.2; no longer R26.2
- net N$12: now also R14.1, R17.2; no longer R13.1, R16.2
- net N$13: now also R9.1; no longer R11.1
- net N$14: now also R18.1; no longer R17.1
- net N$29: now also C22.1, R13.1, R14.2, R9.2; no longer C21.1, R11.2, R12.1, R13.2
- net N$3: now also C24.1, R20.1, R25.2; no longer C23.1, R19.1, R23.2
- net N$45: now also R17.1, R18.2; no longer R16.1, R17.2
- net N$46: now also R10.1; no longer R8.1
- net N$47: now also R26.1; no longer R25.1
- net N$48: now also R10.2; no longer R8.2
- net N$50: now also R23.1; no longer R21.1
- net N$51: now also R23.2, R25.1; no longer R21.2, R23.1
- net N$52: now also R15.1; no longer R14.1
- net N$53: now also R15.2, R16.1; no longer R14.2, R15.1
- net N$55: now also C20.1, R11.2, R12.1, R16.2; no longer C19.1, R10.1, R15.2, R9.2
- net N$58: now also R19.2, R29.1; no longer R18.2, R28.1
- net N$60: now also R27.1; no longer R26.1
- net N$62: now also R26.2; no longer R25.2
- net N$63: now also R19.1; no longer R18.1
- net N$65: now also R30.1; no longer R29.1
- net N$67: now also C32.C; no longer C31.C
- net N$68: now also C32.A, R33.2; no longer C31.A, R32.2
- net N$69: now also C25.1; no longer C24.1
- net N$70: now also C30.1, R28.1, R30.2; no longer C29.1, R27.1, R28.2
- net N$71: now also R21.1; no longer R20.1
- net N$72: now also R32.1; no longer R30.1
- net N$73: now also C31.2, R31.2; no longer C30.2, R30.2
- net N$75: now also C31.1, R32.2, R33.1; no longer C30.1, R31.2, R32.1
- net PARAM1_CV: now also C24.2, R20.2; no longer C23.2, R19.2
- net PARAM2_CV: now also C30.2, R28.2; no longer C29.2, R27.2
- net PD1-XTAL: now also C7.2; no longer C6.2
- net PITCH_CV: now also C22.2, R13.2; no longer C21.2, R12.2
- net RESET: now also C4.1, H2.10, R1.2; no longer H1.10, R2.1, S2.B1, S2.B2
- net RX: now also H3.1, R2.2; no longer H2.4, U1.31
- net TX: now also H3.2, R3.2; no longer H2.5, U1.30
Routing:
- net BOOT_FLASH: track 38.3 -> 0.00 mm, vias 2 -> 0
- net JTCK: track 23.3 -> 0.00 mm, vias 2 -> 0
- net JTDO: track 22.4 -> 0.00 mm, vias 2 -> 0
- net TX: track 28.0 -> 6.47 mm
- net JTDO/SWO: track 0.00 -> 19.5 mm, vias 0 -> 2
- net PARAM1_CV: track 81.3 -> 62.6 mm, vias 4 -> 2
- net RESET: track 47.6 -> 29.9 mm, vias 4 -> 3
- net PARAM2_CV: track 102.0 -> 84.5 mm
- net RX: track 23.2 -> 6.16 mm
- net PITCH_CV: track 69.7 -> 53.1 mm
- net JTCK/SWCLK: track 0.00 -> 16.3 mm
- net JTMS/SWDIO: track 0.00 -> 15.5 mm
- net FM_CV: track 74.4 -> 58.9 mm
- net 12V_U5: track 9.52 -> 24.2 mm
- net TX_R: track 0.00 -> 12.2 mm
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Other:
- board text added: "2020-02-07"
- board text added: "Board derived from work by Émilie Gillet of Mutable Instruments, Magpie Modular, and Neutron Sound"
- board text added: "MAIN BOARD"
- board text added: "SWD/JTAG"
- board text added: "TD-UBSE-F-MB"
- board text added: "tall-dog.com"
- board text added: "µBraids SE"
- board text added: "µBraids SE Main Board TD-UBSE-F-MB CC BY-SA 4.0 2020-02-07 tall-dog.com"
- board text removed: "2018-04-27"
- board text removed: "BOOT"
- board text removed: "Board derived from work by Olivier Gillet of Mutable Instruments, Magpie Modular, and Neutron Sound"
- board text removed: "FTDI"
- board text removed: "GN"
- board text removed: "JTAG"
- board text removed: "RESET"
- board text removed: "TALL-DOG.COM"
- board text removed: "TD-UBSE-E-MB"
- board text removed: "µBraids SE Main Board TD-UBSE-E-MB CC BY-SA 4.0 2018-04-27 tall-dog.com"
- board text removed: "µBraids_SE"
