File: uBraids_SE_Main_Board.sch (EAGLE design)
At the start: 95 parts, among them J1 JACK-THONKICONN, J2 JACK-THONKICONN, J3 JACK-THONKICONN, J4 JACK-THONKICONN, J5 JACK-THONKICONN, J6 JACK-THONKICONN, P1 10kB, P2 10kB, P3 10kB, P4 10kB, P5 10kB, P6 10kB, Q1 MMBT3904, U1 STM32F103-LQFP-48, U2 DAC8551-VSSOP-8, U3 LM4040B25, U4 MCP3204-TSSOP-14, U5 LM1117-3.3, U6 LM4040B10, U7 MCP6004, U8 TL074-TSSOP-14, U9 TL072, X1 8MHz

Commit message: revision C first pass, primarily to address rail clearance
Parts:
- R4: device uBraids_SE:RESISTOR-1206 -> uBraids_SE:RESISTOR-0805
Other:
- note added: "C"
- note added: "Licensed: CC BY-SA 4.0, Board derived from work by: Olivier Gillet of Mutable Instruments, Magpie Modular, and Neutron Sound"
- note removed: "B"
- note removed: "Licensed: CC BY-SA 4.0 Board derived from work by: Olivier Gillet, Magpie Modular, Jim Matheson, and altitude909"
Changed lines of the file:
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@@
 <?xml version="1.0" encoding="utf-8"?>
 <!DOCTYPE eagle SYSTEM "eagle.dtd">
-<eagle version="8.2.1">
+<eagle version="8.4.0">
 <drawing>
 <settings>
 <setting alwaysvectorfont="yes"/>
+<setting keepoldvectorfont="yes"/>
 <setting verticaltext="up"/>
 </settings>
@@
 <part name="D2" library="uBraids_SE" deviceset="DIODE" device="-SOD123" value="1N5819HW"/>
 <part name="H3" library="uBraids_SE" deviceset="HEADER-2X5" device="-PTH-0.1-SHROUDED"/>
-<part name="R4" library="uBraids_SE" deviceset="RESISTOR" device="-1206" value="4.7R"/>
+<part name="R4" library="uBraids_SE" deviceset="RESISTOR" device="-0805" value="4.7R"/>
 <part name="U6" library="uBraids_SE" deviceset="LM4041" device="-SOT-23" value="LM4040B10"/>
 <part name="R7" library="uBraids_SE" deviceset="RESISTOR" device="-1206" value="330R"/>
@@
 <sheet>
 <plain>
-<text x="148.59" y="24.13" size="2.54" layer="94">Licensed: CC BY-SA 4.0
-Board derived from work by: Olivier Gillet,
-Magpie Modular, Jim Matheson, and altitude909</text>
+<text x="148.59" y="24.13" size="2.54" layer="94">Licensed: CC BY-SA 4.0, Board derived from
+work by: Olivier Gillet of Mutable Instruments,
+Magpie Modular, and Neutron Sound</text>
 <text x="148.59" y="6.35" size="2.54" layer="94">Website: TALL-DOG.COM</text>
-<text x="236.22" y="6.35" size="3.81" layer="94">B</text>
+<text x="236.22" y="6.35" size="3.81" layer="94">C</text>
 <text x="186.69" y="11.43" size="2.54" layer="94">N/A</text>
 <text x="247.65" y="19.05" size="3.81" layer="94" align="center-right">Digital</text>
@@
 <sheet>
 <plain>
-<text x="148.59" y="24.13" size="2.54" layer="94">Licensed: CC BY-SA 4.0
-Board derived from work by: Olivier Gillet,
-Magpie Modular, Jim Matheson, and altitude909</text>
+<text x="148.59" y="24.13" size="2.54" layer="94">Licensed: CC BY-SA 4.0, Board derived from
+work by: Olivier Gillet of Mutable Instruments,
+Magpie Modular, and Neutron Sound</text>
 <text x="148.59" y="6.35" size="2.54" layer="94">Website: TALL-DOG.COM</text>
-<text x="236.22" y="6.35" size="3.81" layer="94">B</text>
+<text x="236.22" y="6.35" size="3.81" layer="94">C</text>
 <text x="247.65" y="19.05" size="3.81" layer="94" align="center-right">Analog</text>
 <text x="186.69" y="11.43" size="2.54" layer="94">N/A</text>
@@
 </note>
 <note version="8.2" severity="warning">
-Since Version 8.2, Eagle supports online libraries. The ids
+Since Version 8.2, EAGLE supports online libraries. The ids
 of those online libraries will not be understood (or retained)
 with this version.

Commit message: prep for production of revision C
Parts:
- added HOLE1, HOLE2: HOLE, uBraids_SE:HOLE
- R7: device uBraids_SE:RESISTOR-1206 -> uBraids_SE:RESISTOR-0805
Changed lines of the file:
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@@
 <part name="R4" library="uBraids_SE" deviceset="RESISTOR" device="-0805" value="4.7R"/>
 <part name="U6" library="uBraids_SE" deviceset="LM4041" device="-SOT-23" value="LM4040B10"/>
-<part name="R7" library="uBraids_SE" deviceset="RESISTOR" device="-1206" value="330R"/>
+<part name="R7" library="uBraids_SE" deviceset="RESISTOR" device="-0805" value="330R"/>
 <part name="C17" library="uBraids_SE" deviceset="CAP-NP" device="-0603" value="100n"/>
 <part name="A1" library="uBraids_SE" deviceset="DISPLAY-MODULE" device=""/>
@@
 <part name="FRAME1" library="frames" library_urn="urn:adsk.eagle:library:229" deviceset="LETTER_L" device=""/>
 <part name="FRAME2" library="frames" library_urn="urn:adsk.eagle:library:229" deviceset="LETTER_L" device=""/>
+<part name="HOLE1" library="uBraids_SE" deviceset="HOLE" device=""/>
+<part name="HOLE2" library="uBraids_SE" deviceset="HOLE" device=""/>
 </parts>
 <sheets>
@@
 <instance part="R7" gate="G$1" x="223.52" y="106.68" rot="R270"/>
 <instance part="C17" gate="G$1" x="231.14" y="96.52" rot="R270"/>
+<instance part="HOLE1" gate="G$1" x="104.14" y="162.56"/>
+<instance part="HOLE2" gate="G$1" x="104.14" y="154.94"/>
 </instances>
 <busses>
@@
 with this version.
 </note>
+<note version="8.3" severity="warning">
+Since Version 8.3, EAGLE supports URNs for individual library
+assets (packages, symbols, and devices). The URNs of those assets
+will not be understood (or retained) with this version.
+</note>
 </compatibility>

Commit message: update for Revision E production
Parts:
- added HOLE3: HOLE, uBraids_SE_Library:HOLE
- added P7: 10kB, uBraids_SE_Library:POT-ALPS-VERT-PS
- A1: device uBraids_SE:DISPLAY-MODULE -> uBraids_SE_Library:DISPLAY-MODULE
- C1, C10, C11, C14, C16, C17, C19, C2, C20, C21, C22, C23, C24, C25, C26, C27, C28, C29, C3, C30, C4, C5, C6, C7, C8, C9: device uBraids_SE:CAP-NP-0603 -> uBraids_SE_Library:CAP-NP-0603
- C12, C13, C15, C18: device uBraids_SE:CAP-P-6.6MM -> uBraids_SE_Library:CAP-P-6.6MM
- C31: device uBraids_SE:CAP-P-4.3MM -> uBraids_SE_Library:CAP-P-4.3MM
- D1, D2: device uBraids_SE:DIODE-SOD123 -> uBraids_SE_Library:DIODE-SOD123
- H1: device uBraids_SE:HEADER-2X5-PTH-0.05-SHROUDED-SMD -> uBraids_SE_Library:HEADER-2X5-PTH-0.05-SHROUDED-SMD
- H2: device uBraids_SE:HEADER-1X6-PTH-SHROUDED -> uBraids_SE_Library:HEADER-1X6-PTH-SHROUDED
- H3: device uBraids_SE:HEADER-2X5-PTH-0.1-SHROUDED -> uBraids_SE_Library:HEADER-2X5-PTH-0.1-SHROUDED
- HOLE1, HOLE2: device uBraids_SE:HOLE -> uBraids_SE_Library:HOLE
- J1, J2, J3, J4, J5, J6: device uBraids_SE:JACK-THONKICONN -> uBraids_SE_Library:JACK-THONKICONN
- P1, P2, P3, P4, P5, P6: device uBraids_SE:POT-ALPS-VERT-PS -> uBraids_SE_Library:POT-ALPS-VERT-PS
- Q1: device uBraids_SE:NPN-SOT23-BEC -> uBraids_SE_Library:NPN-SOT23-BEC
- R1, R10, R11, R12, R13, R14, R15, R16, R17, R18, R19, R2, R20, R21, R22, R23, R24, R25, R26, R27, R28, R29, R3, R30, R31, R32, R5, R6, R8, R9: device uBraids_SE:RESISTOR-0603 -> uBraids_SE_Library:RESISTOR-0603
- R4, R7: device uBraids_SE:RESISTOR-0805 -> uBraids_SE_Library:RESISTOR-0805
- S1, S2: device uBraids_SE:SPST-EVQQ2 -> uBraids_SE_Library:SPST-EVQQ2
- S3: device uBraids_SE:ENCODER-SW -> uBraids_SE_Library:ENCODER-SW
- U1: device uBraids_SE:STM32F103-LQFP-48 -> uBraids_SE_Library:STM32F103-LQFP-48
- U2: device uBraids_SE:DAC8551-VSSOP-8 -> uBraids_SE_Library:DAC8551-VSSOP-8
- U3, U6: device uBraids_SE:LM4041-SOT-23 -> uBraids_SE_Library:LM4041-SOT-23
- U4: device uBraids_SE:MCP3204-TSSOP-14 -> uBraids_SE_Library:MCP3204-TSSOP-14
- U5: device uBraids_SE:LM1117-WSON-8 -> uBraids_SE_Library:LM1117-SOT-223
- U7, U8: device uBraids_SE:TL074-TSSOP-14 -> uBraids_SE_Library:TL074-TSSOP-14
- U9: device uBraids_SE:TL072-TSSOP-8 -> uBraids_SE_Library:TL072-TSSOP-8
- X1: device uBraids_SE:CRYSTAL-ABM2 -> uBraids_SE_Library:CRYSTAL-ABM2
Connections:
- removed net N$59: C23.1, P5.A, R19.1, R22.2, R23.2, U7D.-
- new net N$1: P6.S, R26.2
- new net N$3: C23.1, P4.A, R19.1, R22.2, R23.2, U7D.-
- net AREF_-10: now also P5.E, P7.E; no longer P4.E, P6.E
- net GND: now also P5.A, P7.A; no longer P4.A, P6.A
- net N$50: now also P4.E; no longer P5.E
- net N$61: now also P5.S; no longer P4.S
- net N$62: now also P4.S; no longer P5.S
- net N$63: now also P6.E; no longer R26.2
- net N$65: now also P7.S; no longer P6.S
- net N$70: now also P6.A
Other:
- note added: "E"
- note removed: "C"
- moved on the sheet: C29, HOLE1, HOLE2, J5, P4, P5, P6, R18, R26, R27, R28, R29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

Commit message: Revision F
Parts:
- removed A1: DISPLAY-MODULE, uBraids_SE_Library:DISPLAY-MODULE
- removed S2: SPST-EVQQ2, uBraids_SE_Library:SPST-EVQQ2
- removed S3: ENCODER-SW, uBraids_SE_Library:ENCODER-SW
- added C32: 10u, uBraids_SE_Library:CAP-P-4.3MM
- added H4: HEADER-1X5-SSM, uBraids_SE_Library:HEADER-1X5-SSM
- added H5: HEADER-2X5-PTH-0.1-SHROUDED, uBraids_SE_Library:HEADER-2X5-PTH-0.1-SHROUDED
- added R33: 24.9k, uBraids_SE_Library:RESISTOR-0603
- C10, C17, C2, C26, C28, C3, C4, C5: value 100n -> 0.1u
- C11: value 470n -> 0.1u
- C12: value 22uF -> 22u
- C13: value 22uF -> 0.47u; device uBraids_SE_Library:CAP-P-6.6MM -> uBraids_SE_Library:CAP-NP-0603
- C14: value 100n -> 22u; device uBraids_SE_Library:CAP-NP-0603 -> uBraids_SE_Library:CAP-P-6.6MM
- C15, C18: value 47uF -> 0.1u; device uBraids_SE_Library:CAP-P-6.6MM -> uBraids_SE_Library:CAP-NP-0603
- C16: value 100n -> 47u; device uBraids_SE_Library:CAP-NP-0603 -> uBraids_SE_Library:CAP-P-6.6MM
- C19: value 1n -> 47u; device uBraids_SE_Library:CAP-NP-0603 -> uBraids_SE_Library:CAP-P-6.6MM
- C20, C22: value 100n -> 1n
- C21, C23, C29: value 1n -> 0.1u
- C24: value 100p -> 1n
- C25: value 100n -> 100p
- C30: value 47p -> 1n
- C31: value 10uF -> 47p; device uBraids_SE_Library:CAP-P-4.3MM -> uBraids_SE_Library:CAP-NP-0603
- C6: value 18p -> 0.1u
- C7: value 1u -> 18p
- C8: value 100n -> 1u
- H1: value HEADER-2X5-PTH-0.05-SHROUDED-SMD -> HEADER-1X9-SSM; device uBraids_SE_Library:HEADER-2X5-PTH-0.05-SHROUDED-SMD -> uBraids_SE_Library:HEADER-1X9-SSM
- H2: value HEADER-1X6-PTH-SHROUDED -> HEADER-2X5-PTH-0.05-SHROUDED-SMD; device uBraids_SE_Library:HEADER-1X6-PTH-SHROUDED -> uBraids_SE_Library:HEADER-2X5-PTH-0.05-SHROUDED-SMD
- H3: value HEADER-2X5-PTH-0.1-SHROUDED -> HEADER-1X2; device uBraids_SE_Library:HEADER-2X5-PTH-0.1-SHROUDED -> uBraids_SE_Library:HEADER-1X2
- R10, R18, R32: value 24.9k -> 100k
- R11: value 120k -> 200k
- R17, R25: value 100k -> 24.9k
- R19: value 49.9k -> 24.9k
- R2: value 10k -> 100R
- R20: value 39k -> 49.9k
- R21: value 24.9k -> 39k
- R27: value 49.9k -> 100k
- R28: value 24.9k -> 49.9k
- R29: value 200k -> 24.9k
- R3: value 1k -> 100R
- R30: value 1k -> 200k
- R31: value 100k -> 1k
- R4: value 4.7R -> 1k; device uBraids_SE_Library:RESISTOR-0805 -> uBraids_SE_Library:RESISTOR-0603
- R7: value 330R -> 4.7R
- R8: value 100k -> 330R; device uBraids_SE_Library:RESISTOR-0603 -> uBraids_SE_Library:RESISTOR-0805
- R9: value 200k -> 120k
- S1: value SPST-EVQQ2 -> ENCODER-SW; device uBraids_SE_Library:SPST-EVQQ2 -> uBraids_SE_Library:ENCODER-SW
Connections:
- removed net BOOT_FLASH: R1.2, S1.1, U1.BOOT0
- removed net JTCK: H1.4, U1.PA14
- removed net JTDO: H1.6, U1.PB3
- removed net JTMS: H1.2, U1.PA13
- new net JTCK/SWCLK: H2.4, U1.PA14
- new net JTDO/SWO: H2.6, U1.PB3
- new net JTMS/SWDIO: H2.2, U1.PA13
- new net RX_R: R2.1, U1.PA10
- new net TX_R: R3.1, U1.PA9
- net -12V: now also C19.NEG, C29.2, D1.A, R8.1; no longer C18.NEG, C26.2, D2.A, R7.1
- net -12V_BUS: now also D1.C, H5.1, H5.2; no longer D2.C, H3.1, H3.2
- net 12V: now also C16.POS, C23.1, C26.1, D2.C, R7.2; no longer C15.POS, C22.1, C25.1, D1.C, R4.2
- net 12V_BUS: now also D2.A, H5.10, H5.9; no longer D1.A, H3.10, H3.9
- net 12V_U5: now also R7.1; no longer R4.1
- net 3V3: now also C11.1, C14.POS, C15.1, C21.1, C6.1, H2.1, H4.1, R1.1, R4.1; no longer A1.3V3, C13.POS, C14.1, C20.1, C4.1, C7.1, H1.1, R2.2, R3.1, S1.2
- net AREF: now also C13.1, R4.2; no longer C11.1, R3.2
- net AREF_-10: now also C18.1, R11.1, R8.2; no longer C17.1, R7.2, R9.1
- net AUDIO_OUT: now also R21.2; no longer R20.2
- net DISP_CHAR1: now also H1.1; no longer A1.DISP_CHAR1
- net DISP_CHAR2: now also H1.2; no longer A1.DISP_CHAR2
- net DISP_CHAR3: now also H1.6; no longer A1.DISP_CHAR3
- net DISP_CHAR4: now also H1.9; no longer A1.DISP_CHAR4
- net DISP_EN: now also H4.5; no longer A1.DISP_EN
- net DISP_SCK: now also H4.4; no longer A1.DISP_SCK
- net DISP_SER: now also H4.3; no longer A1.DISP_SER
- net ENC_A: now also S1A.B; no longer S3A.B
- net ENC_B: now also S1A.A; no longer S3A.A
- net ENC_CLICK: now also S1B.2; no longer S3B.2
- net FINE_TUNE: now also C17.1; no longer C16.1
- net FM_CV: now also C20.2, R12.2; no longer C19.2, R10.2
- net GND: now also C13.2, C14.NEG, C15.2, C16.NEG, C18.2, C19.POS, C21.2, C23.2, C26.2, C29.1, C6.2, C7.1, H1.4, H1.7, H1.8, H2.3, H2.5, H2.9, H4.2, H5.3, H5.4, H5.5, H5.6, H5.7, H5.8, S1A.C, S1B.1, U1.BOOT0; no longer A1.GND, C13.NEG, C14.2, C15.NEG, C16.2, C18.POS, C20.2, C22.2, C24.2, C26.1, C6.1, C7.2, H1.9, H2.1, H3.3, H3.4, H3.5, H3.6, H3.7, H3.8, R1.1, S2.1, S3A.C, S3B.1
- net JTDI: now also H2.8; no longer H1.8
- net N$1: now also R27.2; no longer R26.2
- net N$12: now also R14.1, R17.2; no longer R13.1, R16.2
- net N$13: now also R9.1; no longer R11.1
- net N$14: now also R18.1; no longer R17.1
- net N$29: now also C22.1, R13.1, R14.2, R9.2; no longer C21.1, R11.2, R12.1, R13.2
- net N$3: now also C24.1, R20.1, R25.2; no longer C23.1, R19.1, R23.2
- net N$45: now also R17.1, R18.2; no longer R16.1, R17.2
- net N$46: now also R10.1; no longer R8.1
- net N$47: now also R26.1; no longer R25.1
- net N$48: now also R10.2; no longer R8.2
- net N$50: now also R23.1; no longer R21.1
- net N$51: now also R23.2, R25.1; no longer R21.2, R23.1
- net N$52: now also R15.1; no longer R14.1
- net N$53: now also R15.2, R16.1; no longer R14.2, R15.1
- net N$55: now also C20.1, R11.2, R12.1, R16.2; no longer C19.1, R10.1, R15.2, R9.2
- net N$58: now also R19.2, R29.1; no longer R18.2, R28.1
- net N$60: now also R27.1; no longer R26.1
- net N$62: now also R26.2; no longer R25.2
- net N$63: now also R19.1; no longer R18.1
- net N$65: now also R30.1; no longer R29.1
- net N$67: now also C32.NEG; no longer C31.NEG
- net N$68: now also C32.POS, R33.2; no longer C31.POS, R32.2
- net N$69: now also C25.1; no longer C24.1
- net N$70: now also C30.1, R28.1, R30.2; no longer C29.1, R27.1, R28.2
- net N$71: now also R21.1; no longer R20.1
- net N$72: now also R32.1; no longer R30.1
- net N$73: now also C31.2, R31.2; no longer C30.2, R30.2
- net N$75: now also C31.1, R32.2, R33.1; no longer C30.1, R31.2, R32.1
- net PARAM1_CV: now also C24.2, R20.2; no longer C23.2, R19.2
- net PARAM2_CV: now also C30.2, R28.2; no longer C29.2, R27.2
- net PD1-XTAL: now also C7.2; no longer C6.2
- net PITCH_CV: now also C22.2, R13.2; no longer C21.2, R12.2
- net RESET: now also C4.1, H2.10, R1.2; no longer H1.10, R2.1, S2.2
- net RX: now also H3.1, R2.2; no longer H2.4, U1.PA10
- net TX: now also H3.2, R3.2; no longer H2.5, U1.PA9
Other:
- note added: "F"
- note added: "Licensed: CC BY-SA 4.0, Board derived from work by: Émilie Gillet of Mutable Instruments, Magpie Modular, and Neutron Sound"
- note added: "Website: tall-dog.com"
- note removed: "E"
- note removed: "Licensed: CC BY-SA 4.0, Board derived from work by: Olivier Gillet of Mutable Instruments, Magpie Modular, and Neutron Sound"
- note removed: "Website: TALL-DOG.COM"
- moved on the sheet: C1, C10, C11, C17, C20, C21, C22, C23, C24, C25, C26, C28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
